File: Pcb/keypad.kicad_pcb (KiCad board)
At the start: 2 copper layers, 75 x 75 mm, 5 parts, among them SW1 SW_Push, SW2 SW_Push, SW3 SW_Push, SW4 SW_Push, U1 MOUDLE-SEEEDUINO-XIAO

Commit message: pcb design
Parts:
- added U2: ER_OLEDM0.91_1x-I2C, Display:ER_OLEDM0.91_1x-I2C, F.Cu at (139.2, 58.0)
- moved SW1 68.8 mm to (106.0, 101.4)
- moved SW4 47.4 mm to (125.0, 82.4)
- moved U1 42.6 mm to (122.5, 66.0)
- moved SW3 33.1 mm to (144.0, 101.5)
- moved SW2 32.7 mm to (125.0, 101.4)
Connections:
- SW1 pad 1: Net-(U1-PA02_A0_D0) -> Net-(U1-PA4_A1_D1)
- SW2 pad 1: Net-(U1-PA4_A1_D1) -> Net-(U1-PA02_A0_D0)
- U1 pad 12: unconnected-(U1-3V3-Pad12) -> Net-(U1-3V3)
- U1 pad 5: unconnected-(U1-PA8_A4_D4_SDA-Pad5) -> Net-(U1-PA8_A4_D4_SDA)
- U1 pad 6: unconnected-(U1-PA9_A5_D5_SCL-Pad6) -> Net-(U1-PA9_A5_D5_SCL)
Routing:
- net Net-(U1-PA8_A4_D4_SDA): track 0.00 -> 93.8 mm
- net GND: track 37.8 -> 106.9 mm
- net Net-(U1-PA11_A3_D3): track 73.9 -> 20.6 mm
- net Net-(U1-PA9_A5_D5_SCL): track 0.00 -> 34.8 mm
- net Net-(U1-PA02_A0_D0): track 29.0 -> 50.4 mm
- net Net-(U1-3V3): track 0.00 -> 14.6 mm
- net Net-(U1-PA4_A1_D1): track 47.6 -> 54.8 mm
- net Net-(U1-PA10_A2_D2): track 46.3 -> 50.1 mm

Commit message: added Cad files and fixed Pcb errors
Routing:
- net Net-(U1-PA4_A1_D1): track 54.8 -> 44.8 mm
- net Net-(U1-PA8_A4_D4_SDA): track 93.8 -> 99.5 mm
- net Net-(U1-PA02_A0_D0): track 50.4 -> 54.5 mm
- net GND: track 106.9 -> 107.8 mm
Changed lines of the file:
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@@
 	)
 	(segment
-		(start 124.96 76.085)
-		(end 124.96 82.42)
-		(width 0.2)
-		(layer "F.Cu")
-		(net "Net-(U1-PA11_A3_D3)")
-	)
-	(segment
-		(start 114.875 66)
-		(end 124.96 76.085)
-		(width 0.2)
-		(layer "F.Cu")
-		(net "Net-(U1-PA11_A3_D3)")
+		(start 121.92 101.42)
+		(end 124.96 101.42)
+		(width 0.2)
+		(layer "F.Cu")
+		(net "Net-(U1-PA02_A0_D0)")
+	)
+	(segment
+		(start 114.875 58.38)
+		(end 113.12 58.38)
+		(width 0.2)
+		(layer "F.Cu")
+		(net "Net-(U1-PA02_A0_D0)")
+	)
+	(segment
+		(start 109.5 89)
+		(end 121.92 101.42)
+		(width 0.2)
+		(layer "F.Cu")
+		(net "Net-(U1-PA02_A0_D0)")
+	)
+	(segment
+		(start 109.5 62)
+		(end 109.5 89)
+		(width 0.2)
+		(layer "F.Cu")
+		(net "Net-(U1-PA02_A0_D0)")
+	)
+	(segment
+		(start 113.12 58.38)
+		(end 109.5 62)
+		(width 0.2)
+		(layer "F.Cu")
+		(net "Net-(U1-PA02_A0_D0)")
+	)
+	(segment
+		(start 130.125 60.92)
+		(end 124.311346 60.92)
+		(width 0.2)
+		(layer "B.Cu")
+		(net "GND")
 	)
 	(segment
@@
 	)
 	(segment
-		(start 111.775 78.125)
-		(end 118.61 84.96)
+		(start 111 71)
+		(end 111 77.35)
 		(width 0.2)
 		(layer "B.Cu")
@@
 	)
 	(segment
+		(start 112.07 69.93)
+		(end 111 71)
+		(width 0.2)
+		(layer "B.Cu")
+		(net "GND")
+	)
+	(segment
 		(start 131.58 60.92)
 		(end 134.5 58)
@@
 	)
 	(segment
-		(start 130.125 60.92)
-		(end 124.311346 60.92)
-		(width 0.2)
-		(layer "B.Cu")
-		(net "GND")
-	)
-	(segment
 		(start 137.69 104)
 		(end 118.65 104)
@@
 	)
 	(segment
+		(start 115.301346 69.93)
+		(end 112.07 69.93)
+		(width 0.2)
+		(layer "B.Cu")
+		(net "GND")
+	)
+	(segment
 		(start 130.125 60.92)
 		(end 131.58 60.92)
@@
 	)
 	(segment
-		(start 112.448654 69.93)
-		(end 111.775 70.603654)
-		(width 0.2)
-		(layer "B.Cu")
-		(net "GND")
-	)
-	(segment
 		(start 118.61 103.96)
 		(end 118.61 84.96)
@@
 	)
 	(segment
-		(start 115.301346 69.93)
-		(end 112.448654 69.93)
-		(width 0.2)
-		(layer "B.Cu")
-		(net "GND")
-	)
-	(segment
-		(start 111.775 70.603654)
-		(end 111.775 78.125)
-		(width 0.2)
-		(layer "B.Cu")
-		(net "GND")
-	)
-	(segment
-		(start 113.838654 58.38)
-		(end 111.775 60.443654)
-		(width 0.2)
-		(layer "F.Cu")
-		(net "Net-(U1-PA02_A0_D0)")
-	)
-	(segment
-		(start 111.775 60.443654)
-		(end 111.775 88.235)
-		(width 0.2)
-		(layer "F.Cu")
-		(net "Net-(U1-PA02_A0_D0)")
-	)
-	(segment
-		(start 111.775 88.235)
-		(end 124.96 101.42)
-		(width 0.2)
-		(layer "F.Cu")
-		(net "Net-(U1-PA02_A0_D0)")
-	)
-	(segment
-		(start 114.875 58.38)
-		(end 113.838654 58.38)
-		(width 0.2)
-		(layer "F.Cu")
-		(net "Net-(U1-PA02_A0_D0)")
-	)
-	(segment
-		(start 115.925 59.87)
-		(end 115.925 57.23)
-		(width 0.2)
-		(layer "F.Cu")
+		(start 111 77.35)
+		(end 118.61 84.96)
+		(width 0.2)
+		(layer "B.Cu")
+		(net "GND")
+	)
+	(segment
+		(start 113.838654 60.92)
+		(end 105.96 68.798654)
+		(width 0.2)
+		(layer "B.Cu")
 		(net "Net-(U1-PA4_A1_D1)")
 	)
 	(segment
-		(start 105.96 63.095)
+		(start 114.875 60.92)
+		(end 113.838654 60.92)
+		(width 0.2)
+		(layer "B.Cu")
+		(net "Net-(U1-PA4_A1_D1)")
+	)
+	(segment
+		(start 105.96 68.798654)
 		(end 105.96 101.42)
 		(width 0.2)
-		(layer "F.Cu")
-		(net "Net-(U1-PA4_A1_D1)")
-	)
-	(segment
-		(start 111.825 57.23)
-		(end 105.96 63.095)
-		(width 0.2)
-		(layer "F.Cu")
-		(net "Net-(U1-PA4_A1_D1)")
-	)
-	(segment
-		(start 115.925 57.23)
-		(end 111.825 57.23)
-		(width 0.2)
-		(layer "F.Cu")
-		(net "Net-(U1-PA4_A1_D1)")
-	)
-	(segment
-		(start 114.875 60.92)
-		(end 115.925 59.87)
-		(width 0.2)
-		(layer "F.Cu")
+		(layer "B.Cu")
 		(net "Net-(U1-PA4_A1_D1)")
 	)
@@
 	)
 	(segment
-		(start 114.875 68.54)
-		(end 116 69.665)
-		(width 0.2)
-		(layer "F.Cu")
-		(net "Net-(U1-PA8_A4_D4_SDA)")
-	)
-	(segment
-		(start 116 75.439899)
-		(end 124.380101 83.82)
-		(width 0.2)
-		(layer "F.Cu")
-		(net "Net-(U1-PA8_A4_D4_SDA)")
-	)
-	(segment
-		(start 143.460101 102.86)
-		(end 144.619899 102.86)
-		(width 0.2)
-		(layer "F.Cu")
-		(net "Net-(U1-PA8_A4_D4_SDA)")
-	)
-	(segment
-		(start 144.619899 102.86)
-		(end 146.81 100.669899)
-		(width 0.2)
-		(layer "F.Cu")
-		(net "Net-(U1-PA8_A4_D4_SDA)")
-	)
-	(segment
-		(start 125.579899 83.82)
-		(end 142.64 100.880101)
-		(width 0.2)
-		(layer "F.Cu")
-		(net "Net-(U1-PA8_A4_D4_SDA)")
-	)
-	(segment
-		(start 142.64 102.039899)
-		(end 143.460101 102.86)
-		(width 0.2)
-		(layer "F.Cu")
-		(net "Net-(U1-PA8_A4_D4_SDA)")
-	)
-	(segment
-		(start 142.64 100.880101)
-		(end 142.64 102.039899)
-		(width 0.2)
-		(layer "F.Cu")
-		(net "Net-(U1-PA8_A4_D4_SDA)")
-	)
-	(segment
-		(start 116 69.665)
-		(end 116 75.439899)
-		(width 0.2)
-		(layer "F.Cu")
-		(net "Net-(U1-PA8_A4_D4_SDA)")
-	)
-	(segment
-		(start 124.380101 83.82)
-		(end 125.579899 83.82)
-		(width 0.2)
-		(layer "F.Cu")
-		(net "Net-(U1-PA8_A4_D4_SDA)")
-	)
-	(segment
-		(start 146.81 100.669899)
-		(end 146.81 58)
-		(width 0.2)
-		(layer "F.Cu")
-		(net "Net-(U1-PA8_A4_D4_SDA)")
+		(start 137.472081 63.46)
+		(end 141.73 59.202081)
+		(width 0.2)
+		(layer "F.Cu")
+		(net "Net-(U1-3V3)")
+	)
+	(segment
+		(start 141.73 59.202081)
+		(end 141.73 58)
+		(width 0.2)
+		(layer "F.Cu")
+		(net "Net-(U1-3V3)")
+	)
+	(segment
+		(start 130.125 63.46)
+		(end 137.472081 63.46)
+		(width 0.2)
+		(layer "F.Cu")
+		(net "Net-(U1-3V3)")
+	)
+	(segment
+		(start 114.875 71.08)
+		(end 115.42 71.08)
+		(width 0.2)
+		(layer "B.Cu")
+		(net "Net-(U1-PA9_A5_D5_SCL)")
+	)
+	(segment
+		(start 115.42 71.08)
+		(end 121.65 64.85)
+		(width 0.2)
+		(layer "B.Cu")
+		(net "Net-(U1-PA9_A5_D5_SCL)")
 	)
 	(segment
@@
 	)
 	(segment
-		(start 121.105 64.85)
+		(start 121.65 64.85)
 		(end 137.42 64.85)
 		(width 0.2)
@@
 	)
 	(segment
-		(start 114.875 71.08)
-		(end 121.105 64.85)
-		(width 0.2)
-		(layer "B.Cu")
-		(net "Net-(U1-PA9_A5_D5_SCL)")
-	)
-	(segment
-		(start 137.472081 63.46)
-		(end 141.73 59.202081)
-		(width 0.2)
-		(layer "F.Cu")
-		(net "Net-(U1-3V3)")
-	)
-	(segment
-		(start 141.73 59.202081)
-		(end 141.73 58)
-		(width 0.2)
-		(layer "F.Cu")
-		(net "Net-(U1-3V3)")
-	)
-	(segment
-		(start 130.125 63.46)
-		(end 137.472081 63.46)
-		(width 0.2)
-		(layer "F.Cu")
-		(net "Net-(U1-3V3)")
+		(start 129 86)
+		(end 138.5 95.5)
+		(width 0.2)
+		(layer "F.Cu")
+		(net "Net-(U1-PA8_A4_D4_SDA)")
+	)
+	(segment
+		(start 139.5 103)
+		(end 146 103)
+		(width 0.2)
+		(layer "F.Cu")
+		(net "Net-(U1-PA8_A4_D4_SDA)")
+	)
+	(segment
+		(start 115.04 68.54)
+		(end 117.5 71)
+		(width 0.2)
+		(layer "F.Cu")
+		(net "Net-(U1-PA8_A4_D4_SDA)")
+	)
+	(segment
+		(start 125 86)
+		(end 129 86)
+		(width 0.2)
+		(layer "F.Cu")
+		(net "Net-(U1-PA8_A4_D4_SDA)")
+	)
+	(segment
+		(start 147.5 101.5)
+		(end 147.5 58.69)
+		(width 0.2)
+		(layer "F.Cu")
+		(net "Net-(U1-PA8_A4_D4_SDA)")
+	)
+	(segment
+		(start 117.5 71)
+		(end 117.5 78.5)
+		(width 0.2)
+		(layer "F.Cu")
+		(net "Net-(U1-PA8_A4_D4_SDA)")
+	)
+	(segment
+		(start 138.5 95.5)
+		(end 138.5 102)
+		(width 0.2)
+		(layer "F.Cu")
+		(net "Net-(U1-PA8_A4_D4_SDA)")
+	)
+	(segment
+		(start 138.5 102)
+		(end 139.5 103)
+		(width 0.2)
+		(layer "F.Cu")
+		(net "Net-(U1-PA8_A4_D4_SDA)")
+	)
+	(segment
+		(start 114.875 68.54)
+		(end 115.04 68.54)
+		(width 0.2)
+		(layer "F.Cu")
+		(net "Net-(U1-PA8_A4_D4_SDA)")
+	)
+	(segment
+		(start 147.5 58.69)
+		(end 146.81 58)
+		(width 0.2)
+		(layer "F.Cu")
+		(net "Net-(U1-PA8_A4_D4_SDA)")
+	)
+	(segment
+		(start 146 103)
+		(end 147.5 101.5)
+		(width 0.2)
+		(layer "F.Cu")
+		(net "Net-(U1-PA8_A4_D4_SDA)")
+	)
+	(segment
+		(start 117.5 78.5)
+		(end 125 86)
+		(width 0.2)
+		(layer "F.Cu")
+		(net "Net-(U1-PA8_A4_D4_SDA)")
+	)
+	(segment
+		(start 114.9375 66)
+		(end 124.96 76.0225)
+		(width 0.2)
+		(layer "F.Cu")
+		(net "Net-(U1-PA11_A3_D3)")
+	)
+	(segment
+		(start 124.96 76.0225)
+		(end 124.96 82.42)
+		(width 0.2)
+		(layer "F.Cu")
+		(net "Net-(U1-PA11_A3_D3)")
+	)
+	(segment
+		(start 114.875 66)
+		(end 114.9375 66)
+		(width 0.2)
+		(layer "F.Cu")
+		(net "Net-(U1-PA11_A3_D3)")
 	)
 	(embedded_fonts no)
