File: Pcb/_restore_backup_2026-06-22T02-33-49-335/keypad.kicad_sch (KiCad schematic)
At the start: 6 parts, among them SW1 SW_Push, SW2 SW_Push, SW3 SW_Push, SW4 SW_Push, U1 MOUDLE-SEEEDUINO-XIAO, U2 ER_OLEDM0.91_1x-I2C

Commit message: worked on pcb
Parts:
- removed U2: ER_OLEDM0.91_1x-I2C, Display:ER_OLEDM0.91_1x-I2C, symbol Display_Graphic:ER_OLEDM0.91_1x-I2C
Connections:
- net at SW1.1: now also U1.1 (PA02_A0_D0); no longer U1.2 (PA4_A1_D1)
- net at SW2.1: now also U1.2 (PA4_A1_D1); no longer U1.1 (PA02_A0_D0)
Other:
- moved on the sheet: SW1, SW2, SW3, SW4, U1
